Commit message: bug fix (#5)
fix view_rv5as
new view_rv2fr
fix rv5as moveit model

File: melfa_description/urdf/rv5as/rv5as.urdf (robot description, URDF)
Before this commit: robot rv5as, 9 links, 8 joints
Links:
- link rv5as_base: geometry collision mesh filename=package://melfa_description/meshes/rv5as/base.STL scale=1 1 1; visual mesh filename=package://melfa_description/meshes/rv5as/base.STL scale=1 1 1
- link rv5as_elbow: geometry collision mesh filename=package://melfa_description/meshes/rv5as/elbow.STL scale=1 1 1; visual mesh filename=package://melfa_description/meshes/rv5as/elbow.STL scale=1 1 1
- link rv5as_forearm: geometry collision mesh filename=package://melfa_description/meshes/rv5as/forearm.STL scale=1 1 1; visual mesh filename=package://melfa_description/meshes/rv5as/forearm.STL scale=1 1 1
- link rv5as_hand_flange: geometry collision mesh filename=package://melfa_description/meshes/rv5as/hand_flange.STL scale=1 1 1; visual mesh filename=package://melfa_description/meshes/rv5as/hand_flange.STL scale=1 1 1
- link rv5as_shoulder: geometry collision mesh filename=package://melfa_description/meshes/rv5as/shoulder.STL scale=1 1 1; visual mesh filename=package://melfa_description/meshes/rv5as/shoulder.STL scale=1 1 1
- link rv5as_upper_arm: geometry collision mesh filename=package://melfa_description/meshes/rv5as/upper_arm.STL scale=1 1 1; visual mesh filename=package://melfa_description/meshes/rv5as/upper_arm.STL scale=1 1 1
- link rv5as_wrist: geometry collision mesh filename=package://melfa_description/meshes/rv5as/wrist.STL scale=1 1 1; visual mesh filename=package://melfa_description/meshes/rv5as/wrist.STL scale=1 1 1
