Commit message: Ver 1.0.3 (#6)
* bug fix

* update readme

* update rv7frl urdf

* update rv7frl mesh files

* update readme

File: melfa_description/urdf/rv7frl/rv7frl.urdf (robot description, URDF)
Before this commit: robot rv7frl, 9 links, 8 joints
Joints:
- removed joint Mate1
- added joint rv7frl_world_to_base: type fixed, parent world, child rv7frl_base, origin xyz=0 0 0 rpy=0 0 0
- joint rv7frl_hand_flange-to-default_tcp: origin xyz=0 0 0 rpy=0 -0 0 -> xyz=0 0 0 rpy=0 0 0
- joint rv7frl_joint_1: origin xyz=0 0 0.224 rpy=0 -0 0 -> xyz=0 0 0 rpy=0 0 0
- joint rv7frl_joint_2: origin xyz=0 0.106 0.176 rpy=0 -0 0 -> xyz=0 0 0.4 rpy=0 0 0
- joint rv7frl_joint_3: origin xyz=0 -0.057 0.435 rpy=0 -0 0 -> xyz=0 0 0.435 rpy=0 0 0
- joint rv7frl_joint_4: origin xyz=-0.05 -0.049 0.1 rpy=0 -0 0 -> xyz=-0.05 0 0 rpy=0 0 0
- joint rv7frl_joint_5: origin xyz=0 -0.021 0.37 rpy=0 -0 0 -> xyz=0 0 0.47 rpy=0 0 0
- joint rv7frl_joint_6: origin xyz=0 0.021 0.085 rpy=0 -0 0 -> xyz=0 0 0.085 rpy=0 0 0

File: melfa_description/urdf/rv7frl/rv7frl_macro.xacro (robot description, xacro)
@@ -5,13 +5,11 @@
             <color rgba="1.0 1.0 1.0 1.0"/>
         </material>
-        <joint name="Mate1" type="fixed">
+        <joint name="rv7frl_world_to_base" type="fixed">
             <origin xyz="0 0 0" rpy="0 -0 0" />
-            <!-- <parent link="world" /> -->
-            <!-- base's praent link -->
             <parent link="${parent}" />
             <child link="rv7frl_base" />
         </joint>
         <joint name="rv7frl_hand_flange-to-default_tcp" type="fixed">
-            <origin xyz="0 0 0" rpy="0 -0 0" />
+            <origin xyz="0 0 0" rpy="0 0 0" />
             <parent link="rv7frl_hand_flange" />
             <child link="rv7frl_default_tcp" />
@@ -20,5 +18,5 @@
             <axis xyz="0 0 1" />
             <limit lower="-4.188790" upper="4.188790" effort="1" velocity="5.026548" />
-            <origin xyz="0 0 0.224" rpy="0 -0 0" />
+            <origin xyz="0 0 0" rpy="0 0 0" />
             <parent link="rv7frl_base" />
             <child link="rv7frl_shoulder" />
@@ -27,5 +25,5 @@
             <axis xyz="0 1 0" />
             <limit lower="-1.919862" upper="2.268928" effort="1" velocity="5.602507" />
-            <origin xyz="0 0.106 0.176" rpy="0 -0 0" />
+            <origin xyz="0 0 0.4" rpy="0 0 0" />
             <parent link="rv7frl_shoulder" />
             <child link="rv7frl_upper_arm" />
@@ -34,5 +32,5 @@
             <axis xyz="0 1 0" />
             <limit lower="0.000000" upper="2.827433" effort="1" velocity="6.283185" />
-            <origin xyz="0 -0.057 0.435" rpy="0 -0 0" />
+            <origin xyz="0 0 0.435" rpy="0 0 0" />
             <parent link="rv7frl_upper_arm" />
             <child link="rv7frl_elbow" />
@@ -41,5 +39,5 @@
             <axis xyz="0 0 1" />
             <limit lower="-3.490659" upper="3.490659" effort="1" velocity="5.881760" />
-            <origin xyz="-0.05 -0.049 0.1" rpy="0 -0 0" />
+            <origin xyz="-0.05 0 0" rpy="0 0 0" />
             <parent link="rv7frl_elbow" />
             <child link="rv7frl_forearm" />
@@ -48,5 +46,5 @@
             <axis xyz="0 1 0" />
             <limit lower="-2.094395" upper="2.094395" effort="1" velocity="7.853981" />
-            <origin xyz="0 -0.021 0.37" rpy="0 -0 0" />
+            <origin xyz="0 0 0.47" rpy="0 0 0" />
             <parent link="rv7frl_forearm" />
             <child link="rv7frl_wrist" />
@@ -55,5 +53,5 @@
             <axis xyz="0 0 1" />
             <limit lower="-6.283185" upper="6.283185" effort="1" velocity="12.566371" />
-            <origin xyz="0 0.021 0.085" rpy="0 -0 0" />
+            <origin xyz="0 0 0.085" rpy="0 0 0" />
             <parent link="rv7frl_wrist" />
             <child link="rv7frl_hand_flange" />
@@ -65,5 +63,5 @@
                     <mesh filename="package://melfa_description/meshes/rv7frl/base.STL" />
                 </geometry>
-                <origin rpy="0.00 0.00 0" xyz="0.00 0.00 0.00"/>
+                <origin rpy="0 0 0" xyz="0 0 0"/>
             </visual>
             <collision>
@@ -71,5 +69,5 @@
                     <mesh filename="package://melfa_description/meshes/rv7frl/base.STL" />
                 </geometry>
-                <origin rpy="0.00 0.00 0" xyz="0.00 0.00 0.00"/>
+                <origin rpy="0 0 0" xyz="0 0 0"/>
             </collision>
         </link>
@@ -81,5 +79,5 @@
                     <mesh filename="package://melfa_description/meshes/rv7frl/elbow.STL" />
                 </geometry>
-                <origin rpy="0.00 0.00 3.14159265359" xyz="0.00 -0.049 0.00"/>
+                <origin rpy="0 0 0" xyz="0 0 0"/>
             </visual>
             <collision>
@@ -87,5 +85,5 @@
                     <mesh filename="package://melfa_description/meshes/rv7frl/elbow.STL" />
                 </geometry>
-                <origin rpy="0.00 0.00 3.14159265359" xyz="0.00 -0.049 0.00"/>
+                <origin rpy="0 0 0" xyz="0 0 0"/>
             </collision>
         </link>
@@ -96,5 +94,5 @@
                     <mesh filename="package://melfa_description/meshes/rv7frl/forearm.STL" />
                 </geometry>
-                <origin rpy="0.00 0.00 0" xyz="0.00 0.00 -0.004"/>
+                <origin rpy="0 0 0" xyz="0 0 0"/>
             </visual>
             <collision>
@@ -102,5 +100,5 @@
                     <mesh filename="package://melfa_description/meshes/rv7frl/forearm.STL" />
                 </geometry>
-                <origin rpy="0.00 0.00 0" xyz="0.00 0.00 -0.004"/>
+                <origin rpy="0 0 0" xyz="0 0 0"/>
             </collision>
         </link>
@@ -111,5 +109,5 @@
                     <mesh filename="package://melfa_description/meshes/rv7frl/hand_flange.STL" />
                 </geometry>
-                <origin rpy="0.00 0.00 0" xyz="0.00 0.00 -0.006"/>
+                <origin rpy="0 0 0" xyz="0 0 0"/>
             </visual>
             <collision>
@@ -117,5 +115,5 @@
                     <mesh filename="package://melfa_description/meshes/rv7frl/hand_flange.STL" />
                 </geometry>
-                <origin rpy="0.00 0.00 0" xyz="0.00 0.00 -0.006"/>
+                <origin rpy="0 0 0" xyz="0 0 0"/>
             </collision>
         </link>
@@ -126,5 +124,5 @@
                     <mesh filename="package://melfa_description/meshes/rv7frl/shoulder.STL" />
                 </geometry>
-                <origin rpy="0.00 0.00 0" xyz="0.00 0.00 0.00"/>
+                <origin rpy="0 0 0" xyz="0 0 0"/>
             </visual>
             <collision>
@@ -132,5 +130,5 @@
                     <mesh filename="package://melfa_description/meshes/rv7frl/shoulder.STL" />
                 </geometry>
-                <origin rpy="0.00 0.00 0" xyz="0.00 0.00 0.00"/>
+                <origin rpy="0 0 0" xyz="0 0 0"/>
             </collision>
         </link>
@@ -141,5 +139,5 @@
                     <mesh filename="package://melfa_description/meshes/rv7frl/upper_arm.STL" />
                 </geometry>
-                <origin rpy="0.00 0.00 0" xyz="0.00 -0.106 0.00"/>
+                <origin rpy="0 0 0" xyz="0 0 0"/>
             </visual>
             <collision>
@@ -147,5 +145,5 @@
                     <mesh filename="package://melfa_description/meshes/rv7frl/upper_arm.STL" />
                 </geometry>
-                <origin rpy="0.00 0.00 0" xyz="0.00 -0.106 0.00"/>
+                <origin rpy="0 0 0" xyz="0 0 0"/>
             </collision>
         </link>
@@ -156,5 +154,5 @@
                     <mesh filename="package://melfa_description/meshes/rv7frl/wrist.STL" />
                 </geometry>
-                <origin rpy="0.00 0.00 0" xyz="0.00 0.021 0.00"/>
+                <origin rpy="0 0 0" xyz="0 0 0"/>
             </visual>
             <collision>
@@ -162,8 +160,7 @@
                     <mesh filename="package://melfa_description/meshes/rv7frl/wrist.STL" />
                 </geometry>
-                <origin rpy="0.00 0.00 0" xyz="0.00 0.021 0.00"/>
+                <origin rpy="0 0 0" xyz="0 0 0"/>
             </collision>
         </link>
-        <!-- <link name="world" /> -->
     </xacro:macro>
 </robot>

File: melfa_moveit_config/melfa_rv7frl_moveit_config/config/rv7frl_macro.srdf.xacro (robot description, xacro)
@@ -19,4 +19,5 @@
             <joint name="rv7frl_joint_6"/>
             <joint name="rv7frl_hand_flange-to-default_tcp"/>
+            <chain base_link="rv7frl_base" tip_link="rv7frl_default_tcp"/>
         </group>
         <!--GROUP STATES: Purpose: Define a named state for a particular group, in terms of joint values. This is useful to define states like 'folded arms'-->
