Commit message: add rv80fr

File: melfa_description/urdf/rv80fr/rv80fr.urdf.xacro (robot description, xacro)
@@ -21,5 +21,5 @@
     <xacro:include filename="$(find melfa_description)/ros2_control/rv80fr.hardware.xacro" />
     <!-- Use world link to fix robot -->
-    <link name="world"/>
+    <link name="$(arg prefix)world"/>
     <xacro:rv80fr parent="$(arg prefix)world" prefix="$(arg prefix)">
         <origin xyz="0 0 0" rpy="0 0 0" />

File: melfa_description/urdf/rv80fr/rv80fr_macro.xacro (robot description, xacro)
@@ -24,5 +24,5 @@
            <joint name="${prefix}rv80fr_world_to_base" type="fixed">
                 <origin rpy="0 0 0" xyz="0 0 0"/>
-                <parent link="${prefix}${parent}"/>
+                <parent link="${parent}"/>
                 <child link="${prefix}rv80fr_base"/>
                 <dynamics damping="1.0" friction="1.0"/>
