Commit message: update melfa_description for gazebo

File: melfa_description/urdf/rv13frl/rv13frl_macro.xacro (robot description, xacro)
@@ -14,5 +14,5 @@
         <xacro:property name="base_mass" value="0.4" />  <!-- These mass are INCORRRECT -->
         <xacro:property name="shoulder_mass" value="0.37000" />
-        <xacro:property name="upper_arm_mass" value="0.83930" />
+        <xacro:property name="upper_arm_mass" value="0.33930" />
         <xacro:property name="elbow_mass" value="0.22750" />
         <xacro:property name="forearm_mass" value="0.12190" />

File: melfa_description/urdf/rv2fr/rv2fr_macro.xacro (robot description, xacro)
@@ -14,9 +14,9 @@
         <xacro:property name="base_mass" value="0.4" />  <!-- These mass are INCORRRECT -->
         <xacro:property name="shoulder_mass" value="0.37000" />
-        <xacro:property name="upper_arm_mass" value="0.83930" />
-        <xacro:property name="elbow_mass" value="0.22750" />
+        <xacro:property name="upper_arm_mass" value="0.33930" />
+        <xacro:property name="elbow_mass" value="0.12190" />
         <xacro:property name="forearm_mass" value="0.12190" />
         <xacro:property name="wrist_mass" value="0.12190" />
-        <xacro:property name="hand_flange_mass" value="0.01879" />
+        <xacro:property name="hand_flange_mass" value="0.12190" />
         <material name="white">
             <color rgba="1.0 1.0 1.0 1.0"/>
@@ -33,5 +33,5 @@
             <child link="${prefix}rv2fr_shoulder"/>
             <axis xyz="0 0 1"/>
-            <limit effort="1" lower="-4.1887902047863905" upper="4.1887902047863905" velocity="5.235987755982989"/>
+            <limit effort="50" lower="-4.1887902047863905" upper="4.1887902047863905" velocity="5.235987755982989"/>
             <dynamics damping="1.0" friction="1.0"/>
         </joint>
@@ -41,5 +41,5 @@
             <child link="${prefix}rv2fr_upper_arm"/>
             <axis xyz="0 1 0"/>
-            <limit effort="1" lower="-2.0943951023931953" upper="2.0943951023931953" velocity="2.6179938779914944"/>
+            <limit effort="50" lower="-2.0943951023931953" upper="2.0943951023931953" velocity="2.6179938779914944"/>
             <dynamics damping="1.0" friction="1.0"/>
         </joint>
@@ -49,5 +49,5 @@
             <child link="${prefix}rv2fr_elbow"/>
             <axis xyz="0 1 0"/>
-            <limit effort="1" lower="0.0" upper="2.792526803190927" velocity="5.235987755982989"/>
+            <limit effort="50" lower="0.0" upper="2.792526803190927" velocity="5.235987755982989"/>
             <dynamics damping="1.0" friction="1.0"/>
         </joint>
@@ -57,5 +57,5 @@
             <child link="${prefix}rv2fr_forearm"/>
             <axis xyz="0 0 1"/>
-            <limit effort="1" lower="-3.490658503988659" upper="3.490658503988659" velocity="7.853981633974483"/>
+            <limit effort="50" lower="-3.490658503988659" upper="3.490658503988659" velocity="7.853981633974483"/>
             <dynamics damping="1.0" friction="1.0"/>
         </joint>
@@ -65,5 +65,5 @@
             <child link="${prefix}rv2fr_wrist"/>
             <axis xyz="0 1 0"/>
-            <limit effort="1" lower="-2.0943951023931953" upper="2.0943951023931953" velocity="7.853981633974483"/>
+            <limit effort="50" lower="-2.0943951023931953" upper="2.0943951023931953" velocity="7.853981633974483"/>
             <dynamics damping="1.0" friction="1.0"/>
         </joint>
@@ -73,5 +73,5 @@
             <child link="${prefix}rv2fr_hand_flange"/>
             <axis xyz="0 0 1"/>
-            <limit effort="1" lower="-6.283185307179586" upper="6.283185307179586" velocity="12.566370614359172"/>
+            <limit effort="50" lower="-6.283185307179586" upper="6.283185307179586" velocity="12.566370614359172"/>
             <dynamics damping="1.0" friction="1.0"/>
         </joint>

File: melfa_description/urdf/rv4fr/rv4fr_macro.xacro (robot description, xacro)
@@ -14,5 +14,5 @@
         <xacro:property name="base_mass" value="0.4" />  <!-- These mass are INCORRRECT -->
         <xacro:property name="shoulder_mass" value="0.37000" />
-        <xacro:property name="upper_arm_mass" value="0.83930" />
+        <xacro:property name="upper_arm_mass" value="0.33930" />
         <xacro:property name="elbow_mass" value="0.22750" />
         <xacro:property name="forearm_mass" value="0.12190" />

File: melfa_description/urdf/rv4frl/rv4frl_macro.xacro (robot description, xacro)
@@ -14,5 +14,5 @@
         <xacro:property name="base_mass" value="0.4" />  <!-- These mass are INCORRRECT -->
         <xacro:property name="shoulder_mass" value="0.37000" />
-        <xacro:property name="upper_arm_mass" value="0.83930" />
+        <xacro:property name="upper_arm_mass" value="0.33930" />
         <xacro:property name="elbow_mass" value="0.22750" />
         <xacro:property name="forearm_mass" value="0.12190" />
@@ -26,5 +26,4 @@
             <parent link="${parent}"/>
             <child link="${prefix}rv4frl_base"/>
-            <dynamics damping="1.0" friction="1.0"/>
         </joint>
         <joint name="${prefix}rv4frl_joint_1" type="revolute">

File: melfa_description/urdf/rv5as/rv5as_macro.xacro (robot description, xacro)
@@ -14,5 +14,5 @@
         <xacro:property name="base_mass" value="0.4" />  <!-- These mass are INCORRRECT -->
         <xacro:property name="shoulder_mass" value="0.37000" />
-        <xacro:property name="upper_arm_mass" value="0.83930" />
+        <xacro:property name="upper_arm_mass" value="0.33930" />
         <xacro:property name="elbow_mass" value="0.22750" />
         <xacro:property name="forearm_mass" value="0.12190" />

File: melfa_description/urdf/rv7frl/rv7frl_macro.xacro (robot description, xacro)
@@ -14,9 +14,10 @@
         <xacro:property name="base_mass" value="0.4" />  <!-- These mass are INCORRRECT -->
         <xacro:property name="shoulder_mass" value="0.37000" />
-        <xacro:property name="upper_arm_mass" value="0.83930" />
-        <xacro:property name="elbow_mass" value="0.22750" />
+        <xacro:property name="upper_arm_mass" value="0.33930" />
+        <xacro:property name="forearm_mass" value="0.22750" />
+        <xacro:property name="elbow_mass" value="0.12190" />
         <xacro:property name="forearm_mass" value="0.12190" />
         <xacro:property name="wrist_mass" value="0.12190" />
-        <xacro:property name="hand_flange_mass" value="0.01879" />
+        <xacro:property name="hand_flange_mass" value="0.12190" />
         <material name="white">
             <color rgba="1.0 1.0 1.0 1.0"/>
@@ -33,5 +34,5 @@
             <child link="${prefix}rv7frl_shoulder"/>
              <axis xyz="0 0 1" />
-            <limit lower="-4.188790" upper="4.188790" effort="1" velocity="5.026548" />
+            <limit lower="-4.188790" upper="4.188790" effort="50" velocity="5.026548" />
             <dynamics damping="1.0" friction="1.0"/>
         </joint>
@@ -41,5 +42,5 @@
             <child link="${prefix}rv7frl_upper_arm"/>
             <axis xyz="0 1 0" />
-            <limit lower="-1.919862" upper="2.268928" effort="1" velocity="5.602507" />
+            <limit lower="-1.919862" upper="2.268928" effort="50" velocity="5.602507" />
             <dynamics damping="1.0" friction="1.0"/>
         </joint>
@@ -49,5 +50,5 @@
             <child link="${prefix}rv7frl_elbow" />
             <axis xyz="0 1 0" />
-            <limit lower="0.000000" upper="2.827433" effort="1" velocity="6.283185" />
+            <limit lower="0.000000" upper="2.827433" effort="50" velocity="6.283185" />
             <dynamics damping="1.0" friction="1.0"/>
         </joint>
@@ -57,5 +58,5 @@
             <child link="${prefix}rv7frl_forearm" />
             <axis xyz="0 0 1" />
-            <limit lower="-3.490659" upper="3.490659" effort="1" velocity="5.881760" />
+            <limit lower="-3.490659" upper="3.490659" effort="50" velocity="5.881760" />
             <dynamics damping="1.0" friction="1.0"/>
         </joint>
@@ -65,5 +66,5 @@
             <child link="${prefix}rv7frl_wrist" />
             <axis xyz="0 1 0" />
-            <limit lower="-2.094395" upper="2.094395" effort="1" velocity="7.853981" />
+            <limit lower="-2.094395" upper="2.094395" effort="50" velocity="7.853981" />
             <dynamics damping="1.0" friction="1.0"/>
         </joint>
@@ -73,5 +74,5 @@
             <child link="${prefix}rv7frl_hand_flange" />
             <axis xyz="0 0 1" />
-            <limit lower="-6.283185" upper="6.283185" effort="1" velocity="12.566371" />
+            <limit lower="-6.283185" upper="6.283185" effort="50" velocity="12.566371" />
             <dynamics damping="1.0" friction="1.0"/>
         </joint>

File: melfa_description/urdf/rv80fr/rv80fr_macro.xacro (robot description, xacro)
@@ -14,9 +14,9 @@
         <xacro:property name="base_mass" value="0.4" />  <!-- These mass are INCORRRECT -->
         <xacro:property name="shoulder_mass" value="0.37000" />
-        <xacro:property name="upper_arm_mass" value="0.83930" />
-        <xacro:property name="elbow_mass" value="0.22750" />
+        <xacro:property name="upper_arm_mass" value="0.33930" />
+        <xacro:property name="elbow_mass" value="0.12190" />
         <xacro:property name="forearm_mass" value="0.12190" />
         <xacro:property name="wrist_mass" value="0.12190" />
-        <xacro:property name="hand_flange_mass" value="0.01879" />
+        <xacro:property name="hand_flange_mass" value="0.12190" />
         <material name="white">
             <color rgba="1.0 1.0 1.0 1.0"/>
@@ -33,5 +33,5 @@
             <child link="${prefix}rv80fr_shoulder"/>
             <axis xyz="0 0 1"/>
-            <limit lower="-3.141592" upper="3.141592" effort="1" velocity="3.141592"/>
+            <limit lower="-3.141592" upper="3.141592" effort="50" velocity="3.141592"/>
             <dynamics damping="1.0" friction="1.0"/>
         </joint>
@@ -41,5 +41,5 @@
             <child link="${prefix}rv80fr_upper_arm"/>
             <axis xyz="0 1 0"/>
-            <limit lower="-1.832596" upper="2.443461" effort="1" velocity="3.141592"/>
+            <limit lower="-1.832596" upper="2.443461" effort="50" velocity="3.141592"/>
             <dynamics damping="1.0" friction="1.0"/>
         </joint>
@@ -49,5 +49,5 @@
             <child link="${prefix}rv80fr_elbow"/>
             <axis xyz="0 1 0"/>
-            <limit lower="-2.356194" upper="2.70526" effort="1" velocity="2.792527"/>
+            <limit lower="-2.356194" upper="2.70526" effort="50" velocity="2.792527"/>
             <dynamics damping="1.0" friction="1.0"/>
         </joint>
@@ -57,5 +57,5 @@
             <child link="${prefix}rv80fr_forearm"/>
             <axis xyz="0 0 1"/>
-            <limit lower="-6.283185" upper="6.283185" effort="1" velocity="3.228859"/>
+            <limit lower="-6.283185" upper="6.283185" effort="50" velocity="3.228859"/>
             <dynamics damping="1.0" friction="1.0"/>
         </joint>
@@ -65,5 +65,5 @@
             <child link="${prefix}rv80fr_wrist"/>
             <axis xyz="0 1 0"/>
-            <limit lower="-2.530727" upper="2.530727" effort="1" velocity="2.879793"/>
+            <limit lower="-2.530727" upper="2.530727" effort="50" velocity="2.879793"/>
             <dynamics damping="1.0" friction="1.0"/>
         </joint>
@@ -73,5 +73,5 @@
             <child link="${prefix}rv80fr_hand_flange"/>
             <axis xyz="0 0 1"/>
-            <limit lower="-7.853982" upper="7.853982" effort="1" velocity="4.886922"/>
+            <limit lower="-7.853982" upper="7.853982" effort="50" velocity="4.886922"/>
             <dynamics damping="1.0" friction="1.0"/>
         </joint>

File: melfa_description/urdf/rv8crl/rv8crl_macro.xacro (robot description, xacro)
@@ -14,5 +14,5 @@
         <xacro:property name="base_mass" value="0.4" />  <!-- These mass are INCORRRECT -->
         <xacro:property name="shoulder_mass" value="0.37000" />
-        <xacro:property name="upper_arm_mass" value="0.83930" />
+        <xacro:property name="upper_arm_mass" value="0.33930" />
         <xacro:property name="elbow_mass" value="0.22750" />
         <xacro:property name="forearm_mass" value="0.12190" />
