Commit message: melfa_description update

File: melfa_description/ros2_control/rh6crh6020.hardware.xacro (robot description, xacro)
@@ -19,4 +19,5 @@
                 <xacro:unless value="${use_fake_hardware or use_sim}">
                     <plugin>melfa_driver/MELFAPositionHardwareInterface</plugin>
+                    <param name="prefix">${prefix}</param>
                     <param name="robot_ip">${robot_ip}</param>
                     <param name="robot_port">${robot_port}</param>
@@ -104,9 +105,9 @@
                     <xacro:gpio_interface interface_name="${prefix}misc3_io" add_state_interfaces="true" add_command_interfaces="true"/>
                 </xacro:if>
-                <gpio name="io_control_mode">
+                <gpio name="${prefix}io_control_mode">
                     <state_interface name="io_mode"/>
                     <command_interface name="io_mode"/>
                 </gpio>
-                <gpio name="ctrl">
+                <gpio name="${prefix}ctrl">
                     <state_interface name="ctrl_type"/>
                     <command_interface name="ctrl_type"/>

File: melfa_description/ros2_control/rh6frh5520.hardware.xacro (robot description, xacro)
@@ -19,4 +19,5 @@
                 <xacro:unless value="${use_fake_hardware or use_sim}">
                     <plugin>melfa_driver/MELFAPositionHardwareInterface</plugin>
+                    <param name="prefix">${prefix}</param>
                     <param name="robot_ip">${robot_ip}</param>
                     <param name="robot_port">${robot_port}</param>
@@ -124,9 +125,9 @@
                     <xacro:gpio_interface interface_name="${prefix}misc3_io" add_state_interfaces="true" add_command_interfaces="true"/>
                 </xacro:if>
-                <gpio name="io_control_mode">
+                <gpio name="${prefix}io_control_mode">
                     <state_interface name="io_mode"/>
                     <command_interface name="io_mode"/>
                 </gpio>
-                <gpio name="ctrl">
+                <gpio name="${prefix}ctrl">
                     <state_interface name="ctrl_type"/>
                     <command_interface name="ctrl_type"/>

File: melfa_description/ros2_control/rv13frl.hardware.xacro (robot description, xacro)
@@ -19,4 +19,5 @@
                 <xacro:unless value="${use_fake_hardware or use_sim}">
                     <plugin>melfa_driver/MELFAPositionHardwareInterface</plugin>
+                    <param name="prefix">${prefix}</param>
                     <param name="robot_ip">${robot_ip}</param>
                     <param name="robot_port">${robot_port}</param>
@@ -48,5 +49,4 @@
                 </command_interface>
                 <state_interface name="position"/>
-                <!-- <state_interface name="velocity"/> -->
             </joint>
             <joint name="${prefix}rv13frl_joint_2">
@@ -141,9 +141,9 @@
                     <xacro:gpio_interface interface_name="${prefix}misc3_io" add_state_interfaces="true" add_command_interfaces="true"/>
                 </xacro:if>
-                <gpio name="io_control_mode">
+                <gpio name="${prefix}io_control_mode">
                     <state_interface name="io_mode"/>
                     <command_interface name="io_mode"/>
                 </gpio>
-                <gpio name="ctrl">
+                <gpio name="${prefix}ctrl">
                     <state_interface name="ctrl_type"/>
                     <command_interface name="ctrl_type"/>

File: melfa_description/ros2_control/rv2fr.hardware.xacro (robot description, xacro)
@@ -19,4 +19,5 @@
                 <xacro:unless value="${use_fake_hardware or use_sim}">
                     <plugin>melfa_driver/MELFAPositionHardwareInterface</plugin>
+                    <param name="prefix">${prefix}</param>
                     <param name="robot_ip">${robot_ip}</param>
                     <param name="robot_port">${robot_port}</param>
@@ -140,9 +141,9 @@
                     <xacro:gpio_interface interface_name="${prefix}misc3_io" add_state_interfaces="true" add_command_interfaces="true"/>
                 </xacro:if>
-                <gpio name="io_control_mode">
+                <gpio name="${prefix}io_control_mode">
                     <state_interface name="io_mode"/>
                     <command_interface name="io_mode"/>
                 </gpio>
-                <gpio name="ctrl">
+                <gpio name="${prefix}ctrl">
                     <state_interface name="ctrl_type"/>
                     <command_interface name="ctrl_type"/>

File: melfa_description/ros2_control/rv4fr.hardware.xacro (robot description, xacro)
@@ -19,4 +19,5 @@
                 <xacro:unless value="${use_fake_hardware or use_sim}">
                     <plugin>melfa_driver/MELFAPositionHardwareInterface</plugin>
+                    <param name="prefix">${prefix}</param>
                     <param name="robot_ip">${robot_ip}</param>
                     <param name="robot_port">${robot_port}</param>
@@ -140,9 +141,9 @@
                     <xacro:gpio_interface interface_name="${prefix}misc3_io" add_state_interfaces="true" add_command_interfaces="true"/>
                 </xacro:if>
-                <gpio name="io_control_mode">
+                <gpio name="${prefix}io_control_mode">
                     <state_interface name="io_mode"/>
                     <command_interface name="io_mode"/>
                 </gpio>
-                <gpio name="ctrl">
+                <gpio name="${prefix}ctrl">
                     <state_interface name="ctrl_type"/>
                     <command_interface name="ctrl_type"/>

File: melfa_description/ros2_control/rv4frl.hardware.xacro (robot description, xacro)
@@ -19,4 +19,5 @@
                 <xacro:unless value="${use_fake_hardware or use_sim}">
                     <plugin>melfa_driver/MELFAPositionHardwareInterface</plugin>
+                    <param name="prefix">${prefix}</param>
                     <param name="robot_ip">${robot_ip}</param>
                     <param name="robot_port">${robot_port}</param>
@@ -140,9 +141,9 @@
                     <xacro:gpio_interface interface_name="${prefix}misc3_io" add_state_interfaces="true" add_command_interfaces="true"/>
                 </xacro:if>
-                <gpio name="io_control_mode">
+                <gpio name="${prefix}io_control_mode">
                     <state_interface name="io_mode"/>
                     <command_interface name="io_mode"/>
                 </gpio>
-                <gpio name="ctrl">
+                <gpio name="${prefix}ctrl">
                     <state_interface name="ctrl_type"/>
                     <command_interface name="ctrl_type"/>

File: melfa_description/ros2_control/rv5as.hardware.xacro (robot description, xacro)
@@ -19,4 +19,5 @@
                 <xacro:unless value="${use_fake_hardware or use_sim}">
                     <plugin>melfa_driver/MELFAPositionHardwareInterface</plugin>
+                    <param name="prefix">${prefix}</param>
                     <param name="robot_ip">${robot_ip}</param>
                     <param name="robot_port">${robot_port}</param>
@@ -120,9 +121,9 @@
                     <xacro:gpio_interface interface_name="${prefix}misc3_io" add_state_interfaces="true" add_command_interfaces="true"/>
                 </xacro:if>
-                <gpio name="io_control_mode">
+                <gpio name="${prefix}io_control_mode">
                     <state_interface name="io_mode"/>
                     <command_interface name="io_mode"/>
                 </gpio>
-                <gpio name="ctrl">
+                <gpio name="${prefix}ctrl">
                     <state_interface name="ctrl_type"/>
                     <command_interface name="ctrl_type"/>

File: melfa_description/ros2_control/rv7frl.hardware.xacro (robot description, xacro)
@@ -19,4 +19,5 @@
                 <xacro:unless value="${use_fake_hardware or use_sim}">
                     <plugin>melfa_driver/MELFAPositionHardwareInterface</plugin>
+                    <param name="prefix">${prefix}</param>
                     <param name="robot_ip">${robot_ip}</param>
                     <param name="robot_port">${robot_port}</param>
@@ -140,9 +141,9 @@
                     <xacro:gpio_interface interface_name="${prefix}misc3_io" add_state_interfaces="true" add_command_interfaces="true"/>
                 </xacro:if>
-                <gpio name="io_control_mode">
+                <gpio name="${prefix}io_control_mode">
                     <state_interface name="io_mode"/>
                     <command_interface name="io_mode"/>
                 </gpio>
-                <gpio name="ctrl">
+                <gpio name="${prefix}ctrl">
                     <state_interface name="ctrl_type"/>
                     <command_interface name="ctrl_type"/>

File: melfa_description/ros2_control/rv80fr.hardware.xacro (robot description, xacro)
@@ -19,4 +19,5 @@
                 <xacro:unless value="${use_fake_hardware or use_sim}">
                     <plugin>melfa_driver/MELFAPositionHardwareInterface</plugin>
+                    <param name="prefix">${prefix}</param>
                     <param name="robot_ip">${robot_ip}</param>
                     <param name="robot_port">${robot_port}</param>
@@ -140,9 +141,9 @@
                     <xacro:gpio_interface interface_name="${prefix}misc3_io" add_state_interfaces="true" add_command_interfaces="true"/>
                 </xacro:if>
-                <gpio name="io_control_mode">
+                <gpio name="${prefix}io_control_mode">
                     <state_interface name="io_mode"/>
                     <command_interface name="io_mode"/>
                 </gpio>
-                <gpio name="ctrl">
+                <gpio name="${prefix}ctrl">
                     <state_interface name="ctrl_type"/>
                     <command_interface name="ctrl_type"/>

File: melfa_description/ros2_control/rv8crl.hardware.xacro (robot description, xacro)
@@ -19,4 +19,5 @@
                 <xacro:unless value="${use_fake_hardware or use_sim}">
                     <plugin>melfa_driver/MELFAPositionHardwareInterface</plugin>
+                    <param name="prefix">${prefix}</param>
                     <param name="robot_ip">${robot_ip}</param>
                     <param name="robot_port">${robot_port}</param>
@@ -120,9 +121,9 @@
                     <xacro:gpio_interface interface_name="${prefix}misc3_io" add_state_interfaces="true" add_command_interfaces="true"/>
                 </xacro:if>
-                <gpio name="io_control_mode">
+                <gpio name="${prefix}io_control_mode">
                     <state_interface name="io_mode"/>
                     <command_interface name="io_mode"/>
                 </gpio>
-                <gpio name="ctrl">
+                <gpio name="${prefix}ctrl">
                     <state_interface name="ctrl_type"/>
                     <command_interface name="ctrl_type"/>

File: melfa_description/urdf/rh6crh6020/rh6crh6020_macro.xacro (robot description, xacro)
@@ -33,5 +33,5 @@
             <child link="${prefix}rh6crh6020_no1arm"/>
             <axis xyz="0 0 1"/>
-            <limit effort="1" lower="-2.303834612632515" upper="2.303834612632515" velocity="7.3303828583761845"/>
+            <limit effort="50" lower="-2.303834612632515" upper="2.303834612632515" velocity="7.3303828583761845"/>
             <dynamics damping="1.0" friction="1.0"/>
         </joint>
@@ -41,5 +41,5 @@
             <child link="${prefix}rh6crh6020_no2arm"/>
             <axis xyz="0 0 1"/>
-            <limit effort="1" lower="-2.6179938779914944" upper="2.6179938779914944" velocity="12.566370614359172"/>
+            <limit effort="50" lower="-2.6179938779914944" upper="2.6179938779914944" velocity="12.566370614359172"/>
             <dynamics damping="1.0" friction="1.0"/>
         </joint>
@@ -49,5 +49,5 @@
             <child link="${prefix}rh6crh6020_shaft_z"/>
             <axis xyz="0 0 1"/>
-            <limit effort="1" lower="-0.051" upper="0.149" velocity="1.1"/>
+            <limit effort="50" lower="-0.051" upper="0.149" velocity="1.1"/>
             <dynamics damping="1.0" friction="1.0"/>
         </joint>
@@ -57,5 +57,5 @@
             <child link="${prefix}rh6crh6020_shaft"/>
             <axis xyz="0 0 1"/>
-            <limit effort="1" lower="-6.283185307179586" upper="6.283185307179586" velocity="43.63323129985824"/>
+            <limit effort="50" lower="-6.283185307179586" upper="6.283185307179586" velocity="43.63323129985824"/>
             <dynamics damping="1.0" friction="1.0"/>
         </joint>

File: melfa_description/urdf/rh6frh5520/rh6frh5520_macro.xacro (robot description, xacro)
@@ -33,5 +33,5 @@
             <child link="${prefix}rh6frh5520_no1arm"/>
             <axis xyz="0 0 1"/>
-            <limit effort="1" lower="-2.9670597283903604" upper="2.9670597283903604" velocity="6.981317007977318"/>
+            <limit effort="50" lower="-2.9670597283903604" upper="2.9670597283903604" velocity="6.981317007977318"/>
             <dynamics damping="1.0" friction="1.0"/>
         </joint>
@@ -41,5 +41,5 @@
             <child link="${prefix}rh6frh5520_no2arm"/>
             <axis xyz="0 0 1"/>
-            <limit effort="1" lower="-2.5307274153917776" upper="2.5307274153917776" velocity="11.693705988362007"/>
+            <limit effort="50" lower="-2.5307274153917776" upper="2.5307274153917776" velocity="11.693705988362007"/>
             <dynamics damping="1.0" friction="1.0"/>
         </joint>
@@ -49,5 +49,5 @@
             <child link="${prefix}rh6frh5520_shaft_z"/>
             <axis xyz="0 0 1"/>
-            <limit effort="1" lower="0.133" upper="0.333" velocity="2.4"/>
+            <limit effort="50" lower="0.133" upper="0.333" velocity="2.4"/>
             <dynamics damping="1.0" friction="1.0"/>
         </joint>
@@ -57,5 +57,5 @@
             <child link="${prefix}rh6frh5520_shaft"/>
             <axis xyz="0 0 1"/>
-            <limit effort="1" lower="-6.283185307179586" upper="6.283185307179586" velocity="43.63323129985824"/>
+            <limit effort="50" lower="-6.283185307179586" upper="6.283185307179586" velocity="43.63323129985824"/>
             <dynamics damping="1.0" friction="1.0"/>
         </joint>

File: melfa_description/urdf/rv13frl/rv13frl_macro.xacro (robot description, xacro)
@@ -33,5 +33,5 @@
             <child link="${prefix}rv13frl_shoulder"/>
             <axis xyz="0 0 1"/>
-            <limit effort="1" lower="-3.3161255787892263" upper="3.3161255787892263" velocity="4.084070449666731"/>
+            <limit effort="50" lower="-3.3161255787892263" upper="3.3161255787892263" velocity="4.084070449666731"/>
             <dynamics damping="1.0" friction="1.0"/>
         </joint>
@@ -41,5 +41,5 @@
             <child link="${prefix}rv13frl_upper_arm"/>
             <axis xyz="0 1 0"/>
-            <limit effort="1" lower="-1.5707963267948966" upper="2.6179938779914944" velocity="2.8623399732707"/>
+            <limit effort="50" lower="-1.5707963267948966" upper="2.6179938779914944" velocity="2.8623399732707"/>
             <dynamics damping="1.0" friction="1.0"/>
         </joint>
@@ -49,5 +49,5 @@
             <child link="${prefix}rv13frl_elbow"/>
             <axis xyz="0 1 0"/>
-            <limit effort="1" lower="-0.17453292519943295" upper="2.748893571891069" velocity="3.822271061867582"/>
+            <limit effort="50" lower="-0.17453292519943295" upper="2.748893571891069" velocity="3.822271061867582"/>
             <dynamics damping="1.0" friction="1.0"/>
         </joint>
@@ -57,5 +57,5 @@
             <child link="${prefix}rv13frl_forearm"/>
             <axis xyz="0 0 1"/>
-            <limit effort="1" lower="-3.490658503988659" upper="3.490658503988659" velocity="6.544984694978735"/>
+            <limit effort="50" lower="-3.490658503988659" upper="3.490658503988659" velocity="6.544984694978735"/>
             <dynamics damping="1.0" friction="1.0"/>
         </joint>
@@ -65,5 +65,5 @@
             <child link="${prefix}rv13frl_wrist"/>
             <axis xyz="0 1 0"/>
-            <limit effort="1" lower="-2.0943951023931953" upper="2.0943951023931953" velocity="6.544984694978735"/>
+            <limit effort="50" lower="-2.0943951023931953" upper="2.0943951023931953" velocity="6.544984694978735"/>
             <dynamics damping="1.0" friction="1.0"/>
         </joint>
@@ -73,5 +73,5 @@
             <child link="${prefix}rv13frl_hand_flange"/>
             <axis xyz="0 0 1"/>
-            <limit effort="1" lower="-6.283185307179586" upper="6.283185307179586" velocity="12.566370614359172"/>
+            <limit effort="50" lower="-6.283185307179586" upper="6.283185307179586" velocity="12.566370614359172"/>
             <dynamics damping="1.0" friction="1.0"/>
         </joint>

File: melfa_description/urdf/rv2fr/rv2fr_macro.xacro (robot description, xacro)
@@ -33,5 +33,5 @@
             <child link="${prefix}rv2fr_shoulder"/>
             <axis xyz="0 0 1"/>
-            <limit effort="50" lower="-4.1887902047863905" upper="4.1887902047863905" velocity="5.235987755982989"/>
+            <limit lower="-4.1887902047863905" upper="4.1887902047863905" effort="50" velocity="5.235987755982989"/>
             <dynamics damping="1.0" friction="1.0"/>
         </joint>
@@ -41,5 +41,5 @@
             <child link="${prefix}rv2fr_upper_arm"/>
             <axis xyz="0 1 0"/>
-            <limit effort="50" lower="-2.0943951023931953" upper="2.0943951023931953" velocity="2.6179938779914944"/>
+            <limit lower="-2.0943951023931953" upper="2.0943951023931953" effort="50" velocity="2.6179938779914944"/>
             <dynamics damping="1.0" friction="1.0"/>
         </joint>
@@ -49,5 +49,5 @@
             <child link="${prefix}rv2fr_elbow"/>
             <axis xyz="0 1 0"/>
-            <limit effort="50" lower="0.0" upper="2.792526803190927" velocity="5.235987755982989"/>
+            <limit lower="0.0" upper="2.792526803190927" effort="500" velocity="5.235987755982989"/>
             <dynamics damping="1.0" friction="1.0"/>
         </joint>
@@ -57,5 +57,5 @@
             <child link="${prefix}rv2fr_forearm"/>
             <axis xyz="0 0 1"/>
-            <limit effort="50" lower="-3.490658503988659" upper="3.490658503988659" velocity="7.853981633974483"/>
+            <limit lower="-3.490658503988659" upper="3.490658503988659" effort="50" velocity="7.853981633974483"/>
             <dynamics damping="1.0" friction="1.0"/>
         </joint>
@@ -65,5 +65,5 @@
             <child link="${prefix}rv2fr_wrist"/>
             <axis xyz="0 1 0"/>
-            <limit effort="50" lower="-2.0943951023931953" upper="2.0943951023931953" velocity="7.853981633974483"/>
+            <limit lower="-2.0943951023931953" upper="2.0943951023931953" effort="50" velocity="7.853981633974483"/>
             <dynamics damping="1.0" friction="1.0"/>
         </joint>
@@ -73,5 +73,5 @@
             <child link="${prefix}rv2fr_hand_flange"/>
             <axis xyz="0 0 1"/>
-            <limit effort="50" lower="-6.283185307179586" upper="6.283185307179586" velocity="12.566370614359172"/>
+            <limit lower="-6.283185307179586" upper="6.283185307179586" effort="50" velocity="12.566370614359172"/>
             <dynamics damping="1.0" friction="1.0"/>
         </joint>

File: melfa_description/urdf/rv4fr/rv4fr_macro.xacro (robot description, xacro)
@@ -33,5 +33,5 @@
             <child link="${prefix}rv4fr_shoulder"/>
             <axis xyz="0 0 1"/>
-            <limit effort="1" lower="-4.1887902047863905" upper="4.1887902047863905" velocity="7.853981633974483"/>
+            <limit effort="50" lower="-4.1887902047863905" upper="4.1887902047863905" velocity="7.853981633974483"/>
             <dynamics damping="1.0" friction="1.0"/>
         </joint>
@@ -41,5 +41,5 @@
             <child link="${prefix}rv4fr_upper_arm"/>
             <axis xyz="0 1 0"/>
-            <limit effort="1" lower="-2.0943951023931953" upper="2.0943951023931953" velocity="7.853981633974483"/>
+            <limit effort="50" lower="-2.0943951023931953" upper="2.0943951023931953" velocity="7.853981633974483"/>
             <dynamics damping="1.0" friction="1.0"/>
         </joint>
@@ -49,5 +49,5 @@
             <child link="${prefix}rv4fr_elbow"/>
             <axis xyz="0 1 0"/>
-            <limit effort="1" lower="0.0" upper="2.8099800957108703" velocity="5.235987755982989"/>
+            <limit effort="50" lower="0.0" upper="2.8099800957108703" velocity="5.235987755982989"/>
             <dynamics damping="1.0" friction="1.0"/>
         </joint>
@@ -57,5 +57,5 @@
             <child link="${prefix}rv4fr_forearm"/>
             <axis xyz="0 0 1"/>
-            <limit effort="1" lower="-3.490658503988659" upper="3.490658503988659" velocity="9.42477796076938"/>
+            <limit effort="50" lower="-3.490658503988659" upper="3.490658503988659" velocity="9.42477796076938"/>
             <dynamics damping="1.0" friction="1.0"/>
         </joint>
@@ -65,5 +65,5 @@
             <child link="${prefix}rv4fr_wrist"/>
             <axis xyz="0 1 0"/>
-            <limit effort="1" lower="-2.0943951023931953" upper="2.0943951023931953" velocity="10.873401239924673"/>
+            <limit effort="50" lower="-2.0943951023931953" upper="2.0943951023931953" velocity="10.873401239924673"/>
             <dynamics damping="1.0" friction="1.0"/>
         </joint>
@@ -73,5 +73,5 @@
             <child link="${prefix}rv4fr_hand_flange"/>
             <axis xyz="0 0 1"/>
-            <limit effort="1" lower="-6.283185307179586" upper="6.283185307179586" velocity="12.566370614359172"/>
+            <limit effort="50" lower="-6.283185307179586" upper="6.283185307179586" velocity="12.566370614359172"/>
             <dynamics damping="1.0" friction="1.0"/>
         </joint>
