Commit message: melfa_description update

File: melfa_description/urdf/rv4frl/rv4frl_macro.xacro (robot description, xacro)
@@ -32,5 +32,5 @@
             <child link="${prefix}rv4frl_shoulder"/>
             <axis xyz="0 0 1"/>
-            <limit effort="1" lower="-4.1887902047863905" upper="4.1887902047863905" velocity="7.3303828583761845"/>
+            <limit effort="50" lower="-4.1887902047863905" upper="4.1887902047863905" velocity="7.3303828583761845"/>
             <dynamics damping="1.0" friction="1.0"/>
         </joint>
@@ -40,5 +40,5 @@
             <child link="${prefix}rv4frl_upper_arm"/>
             <axis xyz="0 1 0"/>
-            <limit effort="1" lower="-2.0943951023931953" upper="2.0943951023931953" velocity="5.8643062867009474"/>
+            <limit effort="50" lower="-2.0943951023931953" upper="2.0943951023931953" velocity="5.8643062867009474"/>
             <dynamics damping="1.0" friction="1.0"/>
         </joint>
@@ -48,5 +48,5 @@
             <child link="${prefix}rv4frl_elbow"/>
             <axis xyz="0 1 0"/>
-            <limit effort="1" lower="0.0" upper="2.8623399732707" velocity="4.363323129985823"/>
+            <limit effort="50" lower="0.0" upper="2.8623399732707" velocity="4.363323129985823"/>
             <dynamics damping="1.0" friction="1.0"/>
         </joint>
@@ -56,5 +56,5 @@
             <child link="${prefix}rv4frl_forearm"/>
             <axis xyz="0 0 1"/>
-            <limit effort="1" lower="-3.490658503988659" upper="3.490658503988659" velocity="9.42477796076938"/>
+            <limit effort="50" lower="-3.490658503988659" upper="3.490658503988659" velocity="9.42477796076938"/>
             <dynamics damping="1.0" friction="1.0"/>
         </joint>
@@ -64,5 +64,5 @@
             <child link="${prefix}rv4frl_wrist"/>
             <axis xyz="0 1 0"/>
-            <limit effort="1" lower="-2.0943951023931953" upper="2.0943951023931953" velocity="10.873401239924673"/>
+            <limit effort="50" lower="-2.0943951023931953" upper="2.0943951023931953" velocity="10.873401239924673"/>
             <dynamics damping="1.0" friction="1.0"/>
         </joint>
@@ -72,5 +72,5 @@
             <child link="${prefix}rv4frl_hand_flange"/>
             <axis xyz="0 0 1"/>
-            <limit effort="1" lower="-6.283185307179586" upper="6.283185307179586" velocity="12.566370614359172"/>
+            <limit effort="50" lower="-6.283185307179586" upper="6.283185307179586" velocity="12.566370614359172"/>
             <dynamics damping="1.0" friction="1.0"/>
         </joint>

File: melfa_description/urdf/rv5as/rv5as.urdf.xacro (robot description, xacro)
@@ -6,5 +6,5 @@
     <xacro:arg name="prefix" default="" />
     <xacro:arg name="robot_ip" default="192.168.0.20" />
-    <xacro:arg name="robot_port" default="10100" />
+    <xacro:arg name="robot_port" default="10000" />
     <xacro:arg name="initial_positions_file" default="initial_positions_rv.yaml" />
     <xacro:arg name="controller_config" default="custom_io_params.yaml" />

File: melfa_description/urdf/rv5as/rv5as_macro.xacro (robot description, xacro)
@@ -33,5 +33,5 @@
             <child link="${prefix}rv5as_shoulder" />
             <axis xyz="0 0 1" />
-            <limit effort="1" velocity="2.16421" lower="-4.18879" upper="4.18879" />
+            <limit effort="50" velocity="2.16421" lower="-4.18879" upper="4.18879" />
             <dynamics damping="1.0" friction="1.0"/>
         </joint>
@@ -41,5 +41,5 @@
             <child link="${prefix}rv5as_upper_arm" />
             <axis xyz="0 1 0" />
-            <limit effort="1" velocity="2.16421" lower="-2.58309" upper="2.58309" />
+            <limit effort="50" velocity="2.16421" lower="-2.58309" upper="2.58309" />
             <dynamics damping="1.0" friction="1.0"/>
         </joint>
@@ -49,5 +49,5 @@
             <child link="${prefix}rv5as_elbow" />
             <axis xyz="0 1 0" />
-            <limit effort="1" velocity="2.16421" lower="-2.61799" upper="2.61799" />
+            <limit effort="50" velocity="2.16421" lower="-2.61799" upper="2.61799" />
             <dynamics damping="1.0" friction="1.0"/>
         </joint>
@@ -57,5 +57,5 @@
             <child link="${prefix}rv5as_forearm" />
             <axis xyz="0 0 1" />
-            <limit effort="1" velocity="3.4383" lower="-3.49066" upper="3.49066" />
+            <limit effort="50" velocity="3.4383" lower="-3.49066" upper="3.49066" />
             <dynamics damping="1.0" friction="1.0"/>
         </joint>
@@ -65,5 +65,5 @@
             <child link="${prefix}rv5as_wrist" />
             <axis xyz="0 1 0" />
-            <limit effort="1" velocity="6.21337" lower="-2.0944" upper="2.0944" />
+            <limit effort="50" velocity="6.21337" lower="-2.0944" upper="2.0944" />
             <dynamics damping="1.0" friction="1.0"/>
         </joint>
@@ -73,5 +73,5 @@
             <child link="${prefix}rv5as_hand_flange" />
             <axis xyz="0 0 1" />
-            <limit effort="1" velocity="6.28318" lower="-3.49066" upper="3.49066" />
+            <limit effort="50" velocity="6.28318" lower="-3.49066" upper="3.49066" />
             <dynamics damping="1.0" friction="1.0"/>
         </joint>

File: melfa_description/urdf/rv8crl/rv8crl_macro.xacro (robot description, xacro)
@@ -33,5 +33,5 @@
             <child link="${prefix}rv8crl_shoulder"/>
             <axis xyz="0 0 1"/>
-            <limit effort="1" lower="-2.9670597283903604" upper="2.9670597283903604" velocity="5.026548245743669"/>
+            <limit effort="50" lower="-2.9670597283903604" upper="2.9670597283903604" velocity="5.026548245743669"/>
             <dynamics damping="1.0" friction="1.0"/>
         </joint>
@@ -41,5 +41,5 @@
             <child link="${prefix}rv8crl_upper_arm"/>
             <axis xyz="0 1 0"/>
-            <limit effort="1" lower="-1.9198621771937625" upper="1.9198621771937625" velocity="5.602506898901797"/>
+            <limit effort="50" lower="-1.9198621771937625" upper="1.9198621771937625" velocity="5.602506898901797"/>
             <dynamics damping="1.0" friction="1.0"/>
         </joint>
@@ -49,5 +49,5 @@
             <child link="${prefix}rv8crl_elbow"/>
             <axis xyz="0 1 0"/>
-            <limit effort="1" lower="0.0" upper="2.8797932657906435" velocity="6.283185307179586"/>
+            <limit effort="50" lower="0.0" upper="2.8797932657906435" velocity="6.283185307179586"/>
             <dynamics damping="1.0" friction="1.0"/>
         </joint>
@@ -57,5 +57,5 @@
             <child link="${prefix}rv8crl_forearm"/>
             <axis xyz="0 0 1"/>
-            <limit effort="1" lower="-3.490658503988659" upper="3.490658503988659" velocity="5.88175957922089"/>
+            <limit effort="50" lower="-3.490658503988659" upper="3.490658503988659" velocity="5.88175957922089"/>
             <dynamics damping="1.0" friction="1.0"/>
         </joint>
@@ -65,5 +65,5 @@
             <child link="${prefix}rv8crl_wrist"/>
             <axis xyz="0 1 0"/>
-            <limit effort="1" lower="-2.0943951023931953" upper="2.0943951023931953" velocity="7.853981633974483"/>
+            <limit effort="50" lower="-2.0943951023931953" upper="2.0943951023931953" velocity="7.853981633974483"/>
             <dynamics damping="1.0" friction="1.0"/>
         </joint>
@@ -73,5 +73,5 @@
             <child link="${prefix}rv8crl_hand_flange"/>
             <axis xyz="0 0 1"/>
-            <limit effort="1" lower="-6.283185307179586" upper="6.283185307179586" velocity="12.566370614359172"/>
+            <limit effort="50" lower="-6.283185307179586" upper="6.283185307179586" velocity="12.566370614359172"/>
             <dynamics damping="1.0" friction="1.0"/>
         </joint>
