Commit message: add launch option to disable packet lost warning message

File: melfa_description/ros2_control/rh6crh6020.hardware.xacro (robot description, xacro)
@@ -1,5 +1,5 @@
 <?xml version="1.0"?>
 <robot xmlns:xacro="http://www.ros.org/wiki/xacro">
-    <xacro:macro name="rh6crh6020_hardware" params="name prefix robot_ip robot_port scara is_j7 j7_linear is_j8 j8_linear initial_positions_file controller_config controller_type use_sim:=^|false use_fake_hardware:=^|true">
+    <xacro:macro name="rh6crh6020_hardware" params="name prefix robot_ip robot_port scara is_j7 j7_linear is_j8 j8_linear packet_lost_log initial_positions_file controller_config controller_type use_sim:=^|false use_fake_hardware:=^|true">
         <xacro:property name="initial_positions" value="${xacro.load_yaml(initial_positions_file)['initial_positions']}"/>
         <xacro:property name="ctrl_limits" value="${xacro.load_yaml(controller_config)['controller_limits']}"/>
@@ -27,4 +27,5 @@
                     <param name="is_j8">${is_j8}</param>
                     <param name="j8_linear">${j8_linear}</param>
+                    <param name="packet_lost_log">${packet_lost_log}</param>
                      <!-- Controller Type R/Q/D -->
                     <param name="controller_type">${controller_type}</param>

File: melfa_description/ros2_control/rh6frh5520.hardware.xacro (robot description, xacro)
@@ -1,5 +1,5 @@
 <?xml version="1.0"?>
 <robot xmlns:xacro="http://www.ros.org/wiki/xacro">
-    <xacro:macro name="rh6frh5520_hardware" params="name prefix robot_ip robot_port scara is_j7 j7_linear is_j8 j8_linear initial_positions_file controller_config controller_type use_sim:=^|false use_fake_hardware:=^|true">
+    <xacro:macro name="rh6frh5520_hardware" params="name prefix robot_ip robot_port scara is_j7 j7_linear is_j8 j8_linear packet_lost_log initial_positions_file controller_config controller_type use_sim:=^|false use_fake_hardware:=^|true">
         <xacro:property name="initial_positions" value="${xacro.load_yaml(initial_positions_file)['initial_positions']}"/>
         <xacro:property name="ctrl_limits" value="${xacro.load_yaml(controller_config)['controller_limits']}"/>
@@ -27,4 +27,5 @@
                     <param name="is_j8">${is_j8}</param>
                     <param name="j8_linear">${j8_linear}</param>
+                    <param name="packet_lost_log">${packet_lost_log}</param>
                      <!-- Controller Type R/Q/D -->
                     <param name="controller_type">${controller_type}</param>

File: melfa_description/ros2_control/rv13frl.hardware.xacro (robot description, xacro)
@@ -1,5 +1,5 @@
 <?xml version="1.0"?>
 <robot xmlns:xacro="http://www.ros.org/wiki/xacro">
-    <xacro:macro name="rv13frl_hardware" params="name prefix robot_ip robot_port scara is_j7 j7_linear is_j8 j8_linear initial_positions_file controller_config controller_type use_sim:=^|false use_fake_hardware:=^|true">
+    <xacro:macro name="rv13frl_hardware" params="name prefix robot_ip robot_port scara is_j7 j7_linear is_j8 j8_linear packet_lost_log initial_positions_file controller_config controller_type use_sim:=^|false use_fake_hardware:=^|true">
         <xacro:property name="initial_positions" value="${xacro.load_yaml(initial_positions_file)['initial_positions']}"/>
         <xacro:property name="ctrl_limits" value="${xacro.load_yaml(controller_config)['controller_limits']}"/>
@@ -27,4 +27,5 @@
                     <param name="is_j8">${is_j8}</param>
                     <param name="j8_linear">${j8_linear}</param>
+                    <param name="packet_lost_log">${packet_lost_log}</param>
                      <!-- Controller Type R/Q/D -->
                     <param name="controller_type">${controller_type}</param>

File: melfa_description/ros2_control/rv2fr.hardware.xacro (robot description, xacro)
@@ -1,5 +1,5 @@
 <?xml version="1.0"?>
 <robot xmlns:xacro="http://www.ros.org/wiki/xacro">
-    <xacro:macro name="rv2fr_hardware" params="name prefix robot_ip robot_port scara is_j7 j7_linear is_j8 j8_linear initial_positions_file controller_config controller_type use_sim:=^|false use_fake_hardware:=^|true">
+    <xacro:macro name="rv2fr_hardware" params="name prefix robot_ip robot_port scara is_j7 j7_linear is_j8 j8_linear packet_lost_log initial_positions_file controller_config controller_type use_sim:=^|false use_fake_hardware:=^|true">
         <xacro:property name="initial_positions" value="${xacro.load_yaml(initial_positions_file)['initial_positions']}"/>
         <xacro:property name="ctrl_limits" value="${xacro.load_yaml(controller_config)['controller_limits']}"/>
@@ -27,4 +27,5 @@
                     <param name="is_j8">${is_j8}</param>
                     <param name="j8_linear">${j8_linear}</param>
+                    <param name="packet_lost_log">${packet_lost_log}</param>
                      <!-- Controller Type R/Q/D -->
                     <param name="controller_type">${controller_type}</param>

File: melfa_description/ros2_control/rv4fr.hardware.xacro (robot description, xacro)
@@ -1,5 +1,5 @@
 <?xml version="1.0"?>
 <robot xmlns:xacro="http://www.ros.org/wiki/xacro">
-    <xacro:macro name="rv4fr_hardware" params="name prefix robot_ip robot_port scara is_j7 j7_linear is_j8 j8_linear initial_positions_file controller_config controller_type use_sim:=^|false use_fake_hardware:=^|true">
+    <xacro:macro name="rv4fr_hardware" params="name prefix robot_ip robot_port scara is_j7 j7_linear is_j8 j8_linear packet_lost_log initial_positions_file controller_config controller_type use_sim:=^|false use_fake_hardware:=^|true">
         <xacro:property name="initial_positions" value="${xacro.load_yaml(initial_positions_file)['initial_positions']}"/>
         <xacro:property name="ctrl_limits" value="${xacro.load_yaml(controller_config)['controller_limits']}"/>
@@ -27,4 +27,5 @@
                     <param name="is_j8">${is_j8}</param>
                     <param name="j8_linear">${j8_linear}</param>
+                    <param name="packet_lost_log">${packet_lost_log}</param>
                      <!-- Controller Type R/Q/D -->
                     <param name="controller_type">${controller_type}</param>

File: melfa_description/ros2_control/rv4frl.hardware.xacro (robot description, xacro)
@@ -1,5 +1,5 @@
 <?xml version="1.0"?>
 <robot xmlns:xacro="http://www.ros.org/wiki/xacro">
-    <xacro:macro name="rv4frl_hardware" params="name prefix robot_ip robot_port scara is_j7 j7_linear is_j8 j8_linear initial_positions_file controller_config controller_type use_sim:=^|false use_fake_hardware:=^|true">
+    <xacro:macro name="rv4frl_hardware" params="name prefix robot_ip robot_port scara is_j7 j7_linear is_j8 j8_linear packet_lost_log initial_positions_file controller_config controller_type use_sim:=^|false use_fake_hardware:=^|true">
         <xacro:property name="initial_positions" value="${xacro.load_yaml(initial_positions_file)['initial_positions']}"/>
         <xacro:property name="ctrl_limits" value="${xacro.load_yaml(controller_config)['controller_limits']}"/>
@@ -27,4 +27,5 @@
                     <param name="is_j8">${is_j8}</param>
                     <param name="j8_linear">${j8_linear}</param>
+                    <param name="packet_lost_log">${packet_lost_log}</param>
                      <!-- Controller Type R/Q/D -->
                     <param name="controller_type">${controller_type}</param>

File: melfa_description/ros2_control/rv5as.hardware.xacro (robot description, xacro)
@@ -1,5 +1,5 @@
 <?xml version="1.0"?>
 <robot xmlns:xacro="http://www.ros.org/wiki/xacro">
-    <xacro:macro name="rv5as_hardware" params="name prefix robot_ip robot_port scara is_j7 j7_linear is_j8 j8_linear initial_positions_file controller_config controller_type use_sim:=^|false use_fake_hardware:=^|true">
+    <xacro:macro name="rv5as_hardware" params="name prefix robot_ip robot_port scara is_j7 j7_linear is_j8 j8_linear packet_lost_log initial_positions_file controller_config controller_type use_sim:=^|false use_fake_hardware:=^|true">
         <xacro:property name="initial_positions" value="${xacro.load_yaml(initial_positions_file)['initial_positions']}"/>
         <xacro:property name="ctrl_limits" value="${xacro.load_yaml(controller_config)['controller_limits']}"/>
@@ -27,4 +27,5 @@
                     <param name="is_j8">${is_j8}</param>
                     <param name="j8_linear">${j8_linear}</param>
+                    <param name="packet_lost_log">${packet_lost_log}</param>
                      <!-- Controller Type R/Q/D -->
                     <param name="controller_type">${controller_type}</param>

File: melfa_description/ros2_control/rv7frl.hardware.xacro (robot description, xacro)
@@ -1,5 +1,5 @@
 <?xml version="1.0"?>
 <robot xmlns:xacro="http://www.ros.org/wiki/xacro">
-    <xacro:macro name="rv7frl_hardware" params="name prefix robot_ip robot_port scara is_j7 j7_linear is_j8 j8_linear initial_positions_file controller_config controller_type use_sim:=^|false use_fake_hardware:=^|true">
+    <xacro:macro name="rv7frl_hardware" params="name prefix robot_ip robot_port scara is_j7 j7_linear is_j8 j8_linear packet_lost_log initial_positions_file controller_config controller_type use_sim:=^|false use_fake_hardware:=^|true">
         <xacro:property name="initial_positions" value="${xacro.load_yaml(initial_positions_file)['initial_positions']}"/>
         <xacro:property name="ctrl_limits" value="${xacro.load_yaml(controller_config)['controller_limits']}"/>
@@ -27,4 +27,5 @@
                     <param name="is_j8">${is_j8}</param>
                     <param name="j8_linear">${j8_linear}</param>
+                    <param name="packet_lost_log">${packet_lost_log}</param>
                      <!-- Controller Type R/Q/D -->
                     <param name="controller_type">${controller_type}</param>

File: melfa_description/ros2_control/rv80fr.hardware.xacro (robot description, xacro)
@@ -1,5 +1,5 @@
 <?xml version="1.0"?>
 <robot xmlns:xacro="http://www.ros.org/wiki/xacro">
-    <xacro:macro name="rv80fr_hardware" params="name prefix robot_ip robot_port scara is_j7 j7_linear is_j8 j8_linear initial_positions_file controller_config controller_type use_sim:=^|false use_fake_hardware:=^|true">
+    <xacro:macro name="rv80fr_hardware" params="name prefix robot_ip robot_port scara is_j7 j7_linear is_j8 j8_linear packet_lost_log initial_positions_file controller_config controller_type use_sim:=^|false use_fake_hardware:=^|true">
         <xacro:property name="initial_positions" value="${xacro.load_yaml(initial_positions_file)['initial_positions']}"/>
         <xacro:property name="ctrl_limits" value="${xacro.load_yaml(controller_config)['controller_limits']}"/>
@@ -27,4 +27,5 @@
                     <param name="is_j8">${is_j8}</param>
                     <param name="j8_linear">${j8_linear}</param>
+                    <param name="packet_lost_log">${packet_lost_log}</param>
                      <!-- Controller Type R/Q/D -->
                     <param name="controller_type">${controller_type}</param>

File: melfa_description/ros2_control/rv8crl.hardware.xacro (robot description, xacro)
@@ -1,5 +1,5 @@
 <?xml version="1.0"?>
 <robot xmlns:xacro="http://www.ros.org/wiki/xacro">
-    <xacro:macro name="rv8crl_hardware" params="name prefix robot_ip robot_port scara is_j7 j7_linear is_j8 j8_linear initial_positions_file controller_config controller_type use_sim:=^|false use_fake_hardware:=^|true">
+    <xacro:macro name="rv8crl_hardware" params="name prefix robot_ip robot_port scara is_j7 j7_linear is_j8 j8_linear packet_lost_log initial_positions_file controller_config controller_type use_sim:=^|false use_fake_hardware:=^|true">
         <xacro:property name="initial_positions" value="${xacro.load_yaml(initial_positions_file)['initial_positions']}"/>
         <xacro:property name="ctrl_limits" value="${xacro.load_yaml(controller_config)['controller_limits']}"/>
@@ -27,4 +27,5 @@
                     <param name="is_j8">${is_j8}</param>
                     <param name="j8_linear">${j8_linear}</param>
+                    <param name="packet_lost_log">${packet_lost_log}</param>
                      <!-- Controller Type R/Q/D -->
                     <param name="controller_type">${controller_type}</param>

File: melfa_description/urdf/rh6crh6020/rh6crh6020.urdf.xacro (robot description, xacro)
@@ -15,4 +15,5 @@
     <xacro:arg name="is_j8" default="0" />
     <xacro:arg name="j8_linear" default="0" />
+    <xacro:arg name="packet_lost_log" default="1" />
     <xacro:arg name="simulation_controllers" default="" />
     <!-- Import urdf file -->
@@ -40,4 +41,5 @@
         use_fake_hardware="$(arg use_fake_hardware)"
         controller_type="$(arg controller_type)"
+        packet_lost_log="$(arg packet_lost_log)"
         />
     <xacro:if value="$(arg use_sim)">

File: melfa_description/urdf/rh6frh5520/rh6frh5520.urdf.xacro (robot description, xacro)
@@ -15,4 +15,5 @@
     <xacro:arg name="is_j8" default="0" />
     <xacro:arg name="j8_linear" default="0" />
+    <xacro:arg name="packet_lost_log" default="1" />
     <xacro:arg name="simulation_controllers" default="" />
     <!-- Import urdf file -->
@@ -40,4 +41,5 @@
         use_fake_hardware="$(arg use_fake_hardware)"
         controller_type="$(arg controller_type)"
+        packet_lost_log="$(arg packet_lost_log)"
         />
     <xacro:if value="$(arg use_sim)">

File: melfa_description/urdf/rv13frl/rv13frl.urdf.xacro (robot description, xacro)
@@ -15,4 +15,5 @@
     <xacro:arg name="is_j8" default="0" />
     <xacro:arg name="j8_linear" default="0" />
+    <xacro:arg name="packet_lost_log" default="1" />
     <xacro:arg name="simulation_controllers" default="" />
     <!-- Import urdf file -->
@@ -40,4 +41,5 @@
         use_fake_hardware="$(arg use_fake_hardware)"
         controller_type="$(arg controller_type)"
+        packet_lost_log="$(arg packet_lost_log)"
         />
         <xacro:if value="$(arg use_sim)">

File: melfa_description/urdf/rv2fr/rv2fr.urdf.xacro (robot description, xacro)
@@ -15,4 +15,5 @@
     <xacro:arg name="is_j8" default="0" />
     <xacro:arg name="j8_linear" default="0" />
+    <xacro:arg name="packet_lost_log" default="1" />
     <xacro:arg name="simulation_controllers" default="" />
     <!-- Import urdf file -->
@@ -40,4 +41,5 @@
         use_fake_hardware="$(arg use_fake_hardware)"
         controller_type="$(arg controller_type)"
+        packet_lost_log="$(arg packet_lost_log)"
         />
     <xacro:if value="$(arg use_sim)">

File: melfa_description/urdf/rv4fr/rv4fr.urdf.xacro (robot description, xacro)
@@ -15,4 +15,5 @@
     <xacro:arg name="is_j8" default="0" />
     <xacro:arg name="j8_linear" default="0" />
+    <xacro:arg name="packet_lost_log" default="1" />
     <xacro:arg name="simulation_controllers" default="" />
     <!-- Import urdf file -->
@@ -40,4 +41,5 @@
         use_fake_hardware="$(arg use_fake_hardware)"
         controller_type="$(arg controller_type)"
+        packet_lost_log="$(arg packet_lost_log)"
         />
     <xacro:if value="$(arg use_sim)">

File: melfa_description/urdf/rv4frl/rv4frl.urdf.xacro (robot description, xacro)
@@ -15,4 +15,5 @@
     <xacro:arg name="is_j8" default="0" />
     <xacro:arg name="j8_linear" default="0" />
+    <xacro:arg name="packet_lost_log" default="1" />
     <xacro:arg name="simulation_controllers" default="" />
     <!-- Import urdf file -->
@@ -40,4 +41,5 @@
         use_fake_hardware="$(arg use_fake_hardware)"
         controller_type="$(arg controller_type)"
+        packet_lost_log="$(arg packet_lost_log)"
         />
         <xacro:if value="$(arg use_sim)">

File: melfa_description/urdf/rv5as/rv5as.urdf.xacro (robot description, xacro)
@@ -15,4 +15,5 @@
     <xacro:arg name="is_j8" default="0" />
     <xacro:arg name="j8_linear" default="0" />
+    <xacro:arg name="packet_lost_log" default="1" />
     <xacro:arg name="simulation_controllers" default="" />
     <!-- Import urdf file -->
@@ -40,4 +41,5 @@
         use_fake_hardware="$(arg use_fake_hardware)"
         controller_type="$(arg controller_type)"
+        packet_lost_log="$(arg packet_lost_log)"
         />
     <xacro:if value="$(arg use_sim)">

File: melfa_description/urdf/rv7frl/rv7frl.urdf.xacro (robot description, xacro)
@@ -15,4 +15,5 @@
     <xacro:arg name="is_j8" default="0" />
     <xacro:arg name="j8_linear" default="0" />
+    <xacro:arg name="packet_lost_log" default="1" />
     <xacro:arg name="simulation_controllers" default="" />
     <!-- Import urdf file -->
@@ -40,4 +41,5 @@
         use_fake_hardware="$(arg use_fake_hardware)"
         controller_type="$(arg controller_type)"
+        packet_lost_log="$(arg packet_lost_log)"
         />
     <xacro:if value="$(arg use_sim)">

File: melfa_description/urdf/rv80fr/rv80fr.urdf.xacro (robot description, xacro)
@@ -15,4 +15,5 @@
     <xacro:arg name="is_j8" default="0" />
     <xacro:arg name="j8_linear" default="0" />
+    <xacro:arg name="packet_lost_log" default="1" />
     <xacro:arg name="simulation_controllers" default="" />
     <!-- Import urdf file -->
@@ -40,4 +41,5 @@
         use_fake_hardware="$(arg use_fake_hardware)"
         controller_type="$(arg controller_type)"
+        packet_lost_log="$(arg packet_lost_log)"
         />
     <xacro:if value="$(arg use_sim)">

File: melfa_description/urdf/rv8crl/rv8crl.urdf.xacro (robot description, xacro)
@@ -15,4 +15,5 @@
     <xacro:arg name="is_j8" default="0" />
     <xacro:arg name="j8_linear" default="0" />
+    <xacro:arg name="packet_lost_log" default="1" />
     <xacro:arg name="simulation_controllers" default="" />
     <!-- Import urdf file -->
@@ -40,4 +41,5 @@
         use_fake_hardware="$(arg use_fake_hardware)"
         controller_type="$(arg controller_type)"
+        packet_lost_log="$(arg packet_lost_log)"
         />
     <xacro:if value="$(arg use_sim)">
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